Commit message: Fix thigh joints: continuous -> revolute with limits (-1.0 to 2.5 rad)

File: resources/robots/aliengo/urdf/aliengo.urdf (robot description, URDF)
Before this commit: robot aliengo_description, 19 links, 18 joints
Joints:
- joint FL_thigh_joint: limit effort=44.4 velocity=40 -> lower=-1.0 upper=2.5 effort=44.4 velocity=40; type continuous -> revolute
- joint FR_thigh_joint: limit effort=44.4 velocity=40 -> lower=-1.0 upper=2.5 effort=44.4 velocity=40; type continuous -> revolute
- joint RL_thigh_joint: limit effort=44.4 velocity=40 -> lower=-1.0 upper=2.5 effort=44.4 velocity=40; type continuous -> revolute
- joint RR_thigh_joint: limit effort=44.4 velocity=40 -> lower=-1.0 upper=2.5 effort=44.4 velocity=40; type continuous -> revolute
